Commit message: Imported upstream version '0.7.1' of 'upstream'

File: fetch_description/robots/fetch.urdf (robot description, URDF)
Before this commit: robot fetch, 26 links, 25 joints
Joints:
- joint laser_joint: origin xyz=0.235 0 0.2878 rpy=3.1415 0 0 -> xyz=0.235 0 0.2878 rpy=3.14159265359 0 0
- joint torso_lift_joint: limit lower=0 upper=0.4 effort=450.0 velocity=0.1 -> lower=0 upper=0.38615 effort=450.0 velocity=0.1

Commit message: Imported upstream version '0.8.1' of 'upstream'

File: fetch_description/robots/fetch.urdf (robot description, URDF)
Before this commit: robot fetch, 26 links, 25 joints
Links:
- link estop_link: geometry collision mesh filename=package://fetch_description/meshes/estop_link.STL; visual mesh filename=package://fetch_description/meshes/estop_link.dae
